File: Schematics/DC-DC_Converter12-400V.sch (KiCad schematic (older format))
At the start: 18 parts

Commit message: Add Schematics Improved .1
Parts:
- removed C?: 2.2nF, symbol Device:C_Small
- removed D? (x2): 1N4001, Diode_THT:D_DO-41_SOD81_P10.16mm_Horizontal, symbol Diode:1N4001
- removed R?: 10k, symbol Device:R_Small
- removed R?: 30, symbol Device:R_Small
- removed U?: IR2153, symbol Driver_FET:IR2153
- added C? (x2): 0.1uF, symbol Device:C_Small
- added D? (x3): 1N5818, Diode_THT:D_DO-41_SOD81_P10.16mm_Horizontal, symbol Diode:1N5818
- added Q? (x2): BC338, Package_TO_SOT_THT:TO-92_Inline, symbol Transistor_BJT:BC338
- added Q? (x2): BC328, Package_TO_SOT_THT:TO-92_Inline, symbol Transistor_BJT:BC328
- added R?: 10, symbol Device:R_Small
- added R? (x4): 1k, symbol Device:R_Small
- added U?: NE555, symbol Timer:NE555
- R?: value 30 -> 10
Connections:
- net GND: now also C?.2, C?.2, Q?.1 (C), Q?.3 (E), U?.1 (GND)
- net +BATT: now reaches BT?.1 (+), C?.1, T?.2 (PM)
- net +BATT: now also Q?.1 (C), Q?.3 (E), R?.1, U?.4 (R), U?.8 (VCC)
- net at R?.1: now also D?.1 (K), Q?.1 (C), Q?.1 (C)
- net at Q?.2 (G): now also D?.2 (A), R?.2
- net at Q?.2 (G), R?.2: now also D?.2 (A)
- new net: C?.1, D?.1 (K), R?.2, U?.2 (TR), U?.6 (THR)
- new net: Q?.2 (B), Q?.2 (B), R?.1, R?.1, U?.3 (Q)
- new net: C?.1, U?.5 (CV)
- new net: D?.2 (A), R?.1, R?.2, U?.7 (DIS)
- new net: D?.1 (K), Q?.3 (E), Q?.3 (E), R?.1
- new net: Q?.2 (B), R?.2 (x2)
Other:
- moved on the sheet: BT?, C?, D?, J?, Q?, R?, T?
